File: Industrial.sch (KiCad schematic (older format))
At the start: 8 parts

Commit message: Finish conecctions
Parts:
- added R? (x6): R, symbol Device:R
- added U3: Esp32, symbol Juanda:Esp32
- J1: renamed from J?; value Screw_Terminal_01x03 -> ASC712
- J2: renamed from J?; value Screw_Terminal_01x06 -> INA219
- gave numbers to parts that had none: 6
Connections:
- net Fase: now reaches L1.1
- net Fase: now also D1.3 (~~), U2.6, R?.2
- net Neutro: now reaches L1.2
- net Neutro: now also D1.4 (~~), R?.2
- net at D1.1 (+): now also Q1.2 (A)
- net GND: now reaches D1.2 (-)
- net GND: now also BT1.2 (-), J1.1 (Pin_1), J2.2 (Pin_2), U1.4, U2.2, R?.2, U3.38 (GND)
- net at Q1.1 (K): now also BT1.1 (+)
- net SCR: now reaches Q1.3 (G)
- net SCR: now also R?.1
- net A0: now reaches J1.2 (Pin_2)
- net A0: now also U3.26 (ADC0)
- net Vcc: now reaches J1.3 (Pin_3)
- net Vcc: now also J2.1 (Pin_1), U3.1 (3.3v)
- net SCL: now reaches J2.3 (Pin_3)
- net SCL: now also U3.36 (SCL)
- net SDA: now reaches J2.4 (Pin_4)
- net SDA: now also U3.33 (SDA)
- net at U1.1: now also R?.1
- net at U1.2: now also R?.1
- net ZeroCross: now reaches U1.5
- net ZeroCross: now also R?.1, U3.24 (ADC2)
- net at U1.6: now also R?.1
- net at U2.1: now also R?.1
- net at U2.4: now also R?.2
- new net 5v: R?.2, U3.19 (5v)
- new net Shoot: R?.2, U3.23 (ADC3)
- no-connect marks 0 -> 32
Other:
- moved on the sheet: BT1, D1, J1, J2, L1, Q1, U1, U2

Commit message: Netlist generated and pcd start
Parts:
- added J3: Corriente, Connector_PinHeader_2.54mm:PinHeader_1x02_P2.54mm_Vertical, symbol Connector:Screw_Terminal_01x02
- added S1: SmithTrigger, Package_DIP:DIP-16_W7.62mm_LongPads, symbol Juanda:SmithTrigger
- BT1, L1: footprint (none) -> TerminalBlock:TerminalBlock_bornier-2_P5.08mm
- D1: footprint (none) -> Diode_THT:Diode_Bridge_Round_D9.0mm
- J1: footprint (none) -> Connector_PinSocket_2.54mm:PinSocket_1x03_P2.54mm_Vertical
- J2: footprint (none) -> Connector_PinSocket_2.54mm:PinSocket_1x06_P2.54mm_Vertical
- R1, R2: renamed from R?; value R -> 1.5K; footprint (none) -> Resistor_THT:R_Axial_DIN0309_L9.0mm_D3.2mm_P5.08mm_Vertical
- R3: renamed from R?; value R -> 100M; footprint (none) -> Resistor_THT:R_Axial_DIN0309_L9.0mm_D3.2mm_P5.08mm_Vertical
- R4: renamed from R?; value R -> 10k; footprint (none) -> Resistor_THT:R_Axial_DIN0309_L9.0mm_D3.2mm_P5.08mm_Vertical
- R5: renamed from R?; value R -> 200; footprint (none) -> Resistor_THT:R_Axial_DIN0309_L9.0mm_D3.2mm_P5.08mm_Vertical
- R6: renamed from R?; value R -> 150; footprint (none) -> Resistor_THT:R_Axial_DIN0309_L9.0mm_D3.2mm_P5.08mm_Vertical
- U1: footprint Package_DIP:DIP-6_W7.62mm -> Package_DIP:DIP-6_W7.62mm_LongPads
- U2: footprint (none) -> Package_DIP:DIP-6_W7.62mm_LongPads
- U3: footprint (none) -> Juanda:ESP32
Connections:
- net GND: now also J3.2 (Pin_2), S1.8 (GND)
- net Vcc: now also S1.1 (Vcc)
- net ZeroCross: now also S1.3 (A); no longer U3.24 (ADC2)
- net Battery: now reaches BT1.1 (+), Q1.1 (K)
- net Battery: now also J3.1 (Pin_1)
- new net TrueZero: S1.4 (notB), U3.24 (ADC2)
- new net notA: S1.2 (notA), S1.5 (B)
- no-connect marks 32 -> 42
Changed lines of the file:
@@
 F 0 "L1" H 2156 4296 50  0000 R CNN
 F 1 "L" H 2156 4205 50  0000 R CNN
-F 2 "" H 2200 4250 50  0001 C CNN
+F 2 "TerminalBlock:TerminalBlock_bornier-2_P5.08mm" H 2200 4250 50  0001 C CNN
 F 3 "~" H 2200 4250 50  0001 C CNN
 	1    2200 4250
@@
 F 0 "D1" H 3250 4500 50  0000 L CNN
 F 1 "D_Bridge_+-AA" H 3200 4600 50  0000 L CNN
-F 2 "" H 3100 4250 50  0001 C CNN
+F 2 "Diode_THT:Diode_Bridge_Round_D9.0mm" H 3100 4250 50  0001 C CNN
 F 3 "~" H 3100 4250 50  0001 C CNN
 	1    3100 4250
@@
 F 0 "J1" V 7022 3030 50  0000 L CNN
 F 1 "ASC712" V 7113 3030 50  0000 L CNN
-F 2 "" H 7150 2850 50  0001 C CNN
+F 2 "Connector_PinSocket_2.54mm:PinSocket_1x03_P2.54mm_Vertical" H 7150 2850 50  0001 C CNN
 F 3 "~" H 7150 2850 50  0001 C CNN
 	1    7150 2850
@@
 F 0 "BT1" H 4768 4546 50  0000 L CNN
 F 1 "Battery_Cell" H 4768 4455 50  0000 L CNN
-F 2 "" V 4650 4510 50  0001 C CNN
+F 2 "TerminalBlock:TerminalBlock_bornier-2_P5.08mm" V 4650 4510 50  0001 C CNN
 F 3 "~" V 4650 4510 50  0001 C CNN
 	1    4650 4450
@@
 F 0 "J2" H 8418 3217 50  0000 C CNN
 F 1 "INA219" H 8418 3126 50  0000 C CNN
-F 2 "" H 8500 2800 50  0001 C CNN
+F 2 "Connector_PinSocket_2.54mm:PinSocket_1x06_P2.54mm_Vertical" H 8500 2800 50  0001 C CNN
 F 3 "~" H 8500 2800 50  0001 C CNN
 	1    8500 2800
@@
 F 0 "U1" H 3000 3325 50  0000 C CNN
 F 1 "H11AA1" H 3000 3234 50  0000 C CNN
-F 2 "Package_DIP:DIP-6_W7.62mm" H 2510 2805 50  0001 L CIN
+F 2 "Package_DIP:DIP-6_W7.62mm_LongPads" H 2510 2805 50  0001 L CIN
 F 3 "https://www.vishay.com/docs/83608/h11aa1.pdf" H 3760 3630 50  0001 L CNN
 	1    3000 3000
@@
 F 0 "U2" H 5550 3175 50  0000 C CNN
 F 1 "MOC3052M" H 5550 3084 50  0000 C CNN
-F 2 "" H 5350 2650 50  0001 L CIN
+F 2 "Package_DIP:DIP-6_W7.62mm_LongPads" H 5350 2650 50  0001 L CIN
 F 3 "https://www.onsemi.com/pub/Collateral/MOC3052M-D.PDF" H 5550 2850 50  0001 L CNN
 	1    5550 2850
@@
 F 0 "U3" H 6775 5715 50  0000 C CNN
 F 1 "Esp32" H 6775 5624 50  0000 C CNN
-F 2 "" H 6450 5350 50  0001 C CNN
+F 2 "Juanda:ESP32" H 6450 5350 50  0001 C CNN
 F 3 "" H 6450 5350 50  0001 C CNN
 	1    6800 4800
@@
 	3400 4250 3850 4250
 $Comp
-L power:GND #PWR?
+L power:GND #PWR02
 U 1 1 6075B7F7
 P 2800 4750
-F 0 "#PWR?" H 2800 4500 50  0001 C CNN
+F 0 "#PWR02" H 2800 4500 50  0001 C CNN
 F 1 "GND" H 2805 4577 50  0000 C CNN
 F 2 "" H 2800 4750 50  0001 C CNN
@@
 $EndComp
 $Comp
-L power:GND #PWR?
+L power:GND #PWR05
 U 1 1 6075BAEC
 P 4650 4700
-F 0 "#PWR?" H 4650 4450 50  0001 C CNN
+F 0 "#PWR05" H 4650 4450 50  0001 C CNN
 F 1 "GND" H 4655 4527 50  0000 C CNN
 F 2 "" H 4650 4700 50  0001 C CNN
@@
 	4650 4550 4650 4700
 $Comp
-L power:GND #PWR?
-U 1 1 6075CB5D
-P 2800 1450
-F 0 "#PWR?" H 2800 1200 50  0001 C CNN
-F 1 "GND" H 2805 1277 50  0000 C CNN
-F 2 "" H 2800 1450 50  0001 C CNN
-F 3 "" H 2800 1450 50  0001 C CNN
-	1    2800 1450
-	1    0    0    -1
-$EndComp
-Text Label 2800 1450 0    50   ~ 0
-GND
-$Comp
-L Device:R R?
+L Device:R R5
 U 1 1 6075D489
 P 4900 2750
-F 0 "R?" V 4693 2750 50  0000 C CNN
-F 1 "R" V 4784 2750 50  0000 C CNN
-F 2 "" V 4830 2750 50  0001 C CNN
+F 0 "R5" V 4693 2750 50  0000 C CNN
+F 1 "200" V 4784 2750 50  0000 C CNN
+F 2 "Resistor_THT:R_Axial_DIN0309_L9.0mm_D3.2mm_P5.08mm_Vertical" V 4830 2750 50  0001 C CNN
 F 3 "~" H 4900 2750 50  0001 C CNN
 	1    4900 2750
@@
 $EndComp
 $Comp
-L Device:R R?
+L Device:R R2
 U 1 1 6075D94A
 P 2400 3100
-F 0 "R?" V 2600 3100 50  0000 C CNN
-F 1 "R" V 2500 3100 50  0000 C CNN
-F 2 "" V 2330 3100 50  0001 C CNN
+F 0 "R2" V 2600 3100 50  0000 C CNN
+F 1 "1.5K" V 2500 3100 50  0000 C CNN
+F 2 "Resistor_THT:R_Axial_DIN0309_L9.0mm_D3.2mm_P5.08mm_Vertical" V 2330 3100 50  0001 C CNN
 F 3 "~" H 2400 3100 50  0001 C CNN
 	1    2400 3100
@@
 $EndComp
 $Comp
-L Device:R R?
+L Device:R R1
 U 1 1 6075DBE5
 P 2400 2900
-F 0 "R?" V 2193 2900 50  0000 C CNN
-F 1 "R" V 2284 2900 50  0000 C CNN
-F 2 "" V 2330 2900 50  0001 C CNN
+F 0 "R1" V 2193 2900 50  0000 C CNN
+F 1 "1.5K" V 2284 2900 50  0000 C CNN
+F 2 "Resistor_THT:R_Axial_DIN0309_L9.0mm_D3.2mm_P5.08mm_Vertical" V 2330 2900 50  0001 C CNN
 F 3 "~" H 2400 2900 50  0001 C CNN
 	1    2400 2900
@@
 $EndComp
 $Comp
-L Device:R R?
+L Device:R R3
 U 1 1 6075E031
 P 3300 2600
-F 0 "R?" H 3230 2554 50  0000 R CNN
-F 1 "R" H 3230 2645 50  0000 R CNN
-F 2 "" V 3230 2600 50  0001 C CNN
+F 0 "R3" H 3230 2554 50  0000 R CNN
+F 1 "100M" H 3230 2645 50  0000 R CNN
+F 2 "Resistor_THT:R_Axial_DIN0309_L9.0mm_D3.2mm_P5.08mm_Vertical" V 3230 2600 50  0001 C CNN
 F 3 "~" H 3300 2600 50  0001 C CNN
 	1    3300 2600
@@
 $EndComp
 $Comp
-L power:GND #PWR?
+L power:GND #PWR04
 U 1 1 6075E57D
 P 3350 3200
-F 0 "#PWR?" H 3350 2950 50  0001 C CNN
+F 0 "#PWR04" H 3350 2950 50  0001 C CNN
 F 1 "GND" H 3355 3027 50  0000 C CNN
 F 2 "" H 3350 3200 50  0001 C CNN
@@
 Wire Wire Line
 	3350 3100 3350 3200
-$Comp
-L power:PWR_FLAG #FLG?
-U 1 1 6075FA1E
-P 2450 1550
-F 0 "#FLG?" H 2450 1625 50  0001 C CNN
-F 1 "PWR_FLAG" H 2450 1723 50  0000 C CNN
-F 2 "" H 2450 1550 50  0001 C CNN
-F 3 "~" H 2450 1550 50  0001 C CNN
-	1    2450 1550
-	1    0    0    -1
-$EndComp
-Text Label 2450 1550 3    50   ~ 0
-5v
 Text Label 6150 5950 2    50   ~ 0
 5v
@@
 	3300 2750 3300 2900
 $Comp
-L power:GND #PWR?
+L power:GND #PWR03
 U 1 1 60762A81
 P 3150 2450
-F 0 "#PWR?" H 3150 2200 50  0001 C CNN
+F 0 "#PWR03" H 3150 2200 50  0001 C CNN
 F 1 "GND" H 3155 2277 50  0000 C CNN
 F 2 "" H 3150 2450 50  0001 C CNN
@@
 5v
 $Comp
-L Device:R R?
+L Device:R R4
 U 1 1 6075E2EE
 P 3700 2750
-F 0 "R?" H 3630 2704 50  0000 R CNN
-F 1 "R" H 3630 2795 50  0000 R CNN
-F 2 "" V 3630 2750 50  0001 C CNN
+F 0 "R4" H 3630 2704 50  0000 R CNN
+F 1 "10k" H 3630 2795 50  0000 R CNN
+F 2 "Resistor_THT:R_Axial_DIN0309_L9.0mm_D3.2mm_P5.08mm_Vertical" V 3630 2750 50  0001 C CNN
 F 3 "~" H 3700 2750 50  0001 C CNN
 	1    3700 2750
@@
 Text Label 3700 3000 0    50   ~ 0
 ZeroCross
-Text Label 7400 5550 0    50   ~ 0
+Text Label 8400 4450 2    50   ~ 0
 ZeroCross
 $Comp
-L power:GND #PWR?
+L power:GND #PWR06
 U 1 1 6077650A
 P 5200 3100
-F 0 "#PWR?" H 5200 2850 50  0001 C CNN
+F 0 "#PWR06" H 5200 2850 50  0001 C CNN
 F 1 "GND" H 5205 2927 50  0000 C CNN
 F 2 "" H 5200 3100 50  0001 C CNN
@@
 Shoot
 $Comp
-L Device:R R?
+L Device:R R6
 U 1 1 60778062
 P 6150 2950
-F 0 "R?" V 5950 2950 50  0000 C CNN
-F 1 "R" V 6050 2950 50  0000 C CNN
-F 2 "" V 6080 2950 50  0001 C CNN
+F 0 "R6" V 5950 2950 50  0000 C CNN
+F 1 "150" V 6050 2950 50  0000 C CNN
+F 2 "Resistor_THT:R_Axial_DIN0309_L9.0mm_D3.2mm_P5.08mm_Vertical" V 6080 2950 50  0001 C CNN
 F 3 "~" H 6150 2950 50  0001 C CNN
 	1    6150 2950
@@
 NoConn ~ 6150 5250
 NoConn ~ 6150 5350
-NoConn ~ 6150 5450
 NoConn ~ 6150 5550
 NoConn ~ 6150 5650
@@
 NoConn ~ 7400 4950
 NoConn ~ 7400 4850
-NoConn ~ 7400 4750
 NoConn ~ 7400 4550
 NoConn ~ 7400 4450
 NoConn ~ 7400 4250
+NoConn ~ 6150 5450
+NoConn ~ 7400 4750
+Text Label 2500 1550 3    50   ~ 0
+Vcc
+$Comp
+L power:PWR_FLAG #FLG0101
+U 1 1 6078F82B
+P 2500 1550
+F 0 "#FLG0101" H 2500 1625 50  0001 C CNN
+F 1 "PWR_FLAG" H 2500 1723 50  0000 C CNN
+F 2 "" H 2500 1550 50  0001 C CNN
+F 3 "~" H 2500 1550 50  0001 C CNN
+	1    2500 1550
+	1    0    0    -1
+$EndComp
+Text Label 2800 1450 0    50   ~ 0
+GND
+$Comp
+L power:GND #PWR01
+U 1 1 6075CB5D
+P 2800 1450
+F 0 "#PWR01" H 2800 1200 50  0001 C CNN
+F 1 "GND" H 2805 1277 50  0000 C CNN
+F 2 "" H 2800 1450 50  0001 C CNN
+F 3 "" H 2800 1450 50  0001 C CNN
+	1    2800 1450
+	1    0    0    -1
+$EndComp
+$Comp
+L Connector:Screw_Terminal_01x02 J3
+U 1 1 607B0D3D
+P 7950 3600
+F 0 "J3" V 8000 3800 50  0000 R CNN
+F 1 "Corriente" V 8100 3850 50  0000 R CNN
+F 2 "Connector_PinHeader_2.54mm:PinHeader_1x02_P2.54mm_Vertical" H 7950 3600 50  0001 C CNN
+F 3 "~" H 7950 3600 50  0001 C CNN
+	1    7950 3600
+	0    -1   1    0
+$EndComp
+Text Label 4650 4250 0    50   ~ 0
+Battery
+Text Label 7950 3400 2    50   ~ 0
+Battery
+$Comp
+L power:GND #PWR07
+U 1 1 607B26DF
+P 8250 3700
+F 0 "#PWR07" H 8250 3450 50  0001 C CNN
+F 1 "GND" H 8255 3527 50  0000 C CNN
+F 2 "" H 8250 3700 50  0001 C CNN
+F 3 "" H 8250 3700 50  0001 C CNN
+	1    8250 3700
+	1    0    0    -1
+$EndComp
+Wire Wire Line
+	8050 3400 8250 3400
+Wire Wire Line
+	8250 3400 8250 3700
+$Comp
+L Juanda:SmithTrigger S1
+U 1 1 607B4B57
+P 8850 4450
+F 0 "S1" H 8850 4915 50  0000 C CNN
+F 1 "SmithTrigger" H 8850 4824 50  0000 C CNN
+F 2 "Package_DIP:DIP-16_W7.62mm_LongPads" H 8850 4450 50  0001 C CNN
+F 3 "" H 8850 4450 50  0001 C CNN
+	1    8850 4450
+	1    0    0    -1
+$EndComp
+Text Label 8400 4250 2    50   ~ 0
+Vcc
+Text Label 8400 4950 2    50   ~ 0
+GND
+Text Label 8400 4350 2    50   ~ 0
+notA
+Text Label 8400 4650 2    50   ~ 0
+notA
+Text Label 8400 4550 2    50   ~ 0
+TrueZero
+Text Label 7400 5550 0    50   ~ 0
+TrueZero
+NoConn ~ 8400 4750
+NoConn ~ 8400 4850
+NoConn ~ 9300 4950
+NoConn ~ 9300 4850
+NoConn ~ 9300 4750
+NoConn ~ 9300 4650
+NoConn ~ 9300 4550
+NoConn ~ 9300 4450
+NoConn ~ 9300 4350
+NoConn ~ 9300 4250
 $EndSCHEMATC

Commit message: finish first version
Parts:
- removed J3: Corriente, Connector_PinHeader_2.54mm:PinHeader_1x02_P2.54mm_Vertical, symbol Connector:Screw_Terminal_01x02
- added J4: Corriente, Connector_PinHeader_2.54mm:PinHeader_1x02_P2.54mm_Vertical, symbol Connector:Screw_Terminal_01x02
- Q1: footprint Package_TO_SOT_THT:TO-220-3_Vertical -> TerminalBlock:TerminalBlock_bornier-3_P5.08mm
Connections:
- net 5v: now also J2.1 (Pin_1), S1.16 (NC)
- net Battery: now also J4.2 (Pin_2); no longer Q1.1 (K)
- net GND: now also U3.32 (GND)
- net Vcc: no longer J2.1 (Pin_1), S1.1 (Vcc)
- net notA: no longer names the net of S1.2 (notA), S1.5 (B)
- new net: J4.1 (Pin_1), Q1.1 (K)
- no-connect marks 42 -> 41
Other:
- note added: "ACS712\nCurrent Sensor\n"
- note added: "ESP32\n"
- note added: "H11AA1 Zero cross"
- note added: "INA219\nVoltaje Sensor\n"
- note added: "MOC3052 Shoot SCR\n"
- note added: "POWER"
- note added: "Secondary transformer and SCR\n"
- note added: "SmithTrigger\n"
- moved on the sheet: J1, J2, R1, R2, R3, R4, R5, R6, U1, U2

Commit message: add rectifier start new desing
Parts:
- added C1: 1000uF, Capacitor_THT:CP_Radial_D13.0mm_P5.00mm, symbol Device:C
- added D2: D, Diode_THT:D_A-405_P7.62mm_Horizontal, symbol Device:D
- added D3: LED, LED_THT:LED_D4.0mm, symbol Device:LED
- added J3: Conn_01x02, Connector_PinHeader_2.54mm:PinHeader_1x02_P2.54mm_Vertical, symbol Connector_Generic:Conn_01x02
- added R7: 440, Resistor_THT:R_Axial_DIN0309_L9.0mm_D3.2mm_P5.08mm_Vertical, symbol Device:R
- added U4: LM7805_TO220, Package_TO_SOT_THT:TO-220-3_Vertical, symbol Regulator_Linear:LM7805_TO220
Connections:
- net 5v: now also J3.1 (Pin_1)
- net GND: now also C1.2, D3.1 (K), U4.2 (GND)
- net bridge: now reaches D1.1 (+), Q1.2 (A)
- net bridge: now also D2.2 (A)
- new net: C1.1, D2.1 (K), U4.1 (VI)
- new net: J3.2 (Pin_2), R7.2, U4.3 (VO)
- new net: D3.2 (A), R7.1
Other:
- note added: "Rectificador AC-DC\n"
Changed lines of the file:
@@
 Text Notes 7500 3650 0    98   ~ 20
 SmithTrigger\n
+$Comp
+L Device:C C1
+U 1 1 607505F1
+P 3000 5950
+F 0 "C1" H 3115 5996 50  0000 L CNN
+F 1 "1000uF" H 3115 5905 50  0000 L CNN
+F 2 "Capacitor_THT:CP_Radial_D13.0mm_P5.00mm" H 3038 5800 50  0001 C CNN
+F 3 "~" H 3000 5950 50  0001 C CNN
+	1    3000 5950
+	1    0    0    -1
+$EndComp
+$Comp
+L Device:D D2
+U 1 1 60751443
+P 2600 5700
+F 0 "D2" H 2600 5483 50  0000 C CNN
+F 1 "D" H 2600 5574 50  0000 C CNN
+F 2 "Diode_THT:D_A-405_P7.62mm_Horizontal" H 2600 5700 50  0001 C CNN
+F 3 "~" H 2600 5700 50  0001 C CNN
+	1    2600 5700
+	-1   0    0    1
+$EndComp
+$Comp
+L Regulator_Linear:LM7805_TO220 U4
+U 1 1 60751E4D
+P 3650 5700
+F 0 "U4" H 3650 5942 50  0000 C CNN
+F 1 "LM7805_TO220" H 3650 5851 50  0000 C CNN
+F 2 "Package_TO_SOT_THT:TO-220-3_Vertical" H 3650 5925 50  0001 C CIN
+F 3 "https://www.onsemi.cn/PowerSolutions/document/MC7800-D.PDF" H 3650 5650 50  0001 C CNN
+	1    3650 5700
+	1    0    0    -1
+$EndComp
+Text Label 3550 4250 3    50   ~ 0
+bridge
+Text Label 2450 5700 2    50   ~ 0
+bridge
+Wire Wire Line
+	2750 5700 3000 5700
+Wire Wire Line
+	3000 5700 3000 5800
+Wire Wire Line
+	3350 5700 3000 5700
+Connection ~ 3000 5700
+Text Label 4450 5700 0    50   ~ 0
+5v
+$Comp
+L Device:R R7
+U 1 1 6075761B
+P 4100 6000
+F 0 "R7" V 3900 6000 50  0000 C CNN
+F 1 "440" V 4000 6000 50  0000 C CNN
+F 2 "Resistor_THT:R_Axial_DIN0309_L9.0mm_D3.2mm_P5.08mm_Vertical" V 4030 6000 50  0001 C CNN
+F 3 "~" H 4100 6000 50  0001 C CNN
+	1    4100 6000
+	1    0    0    1
+$EndComp
+$Comp
+L Device:LED D3
+U 1 1 607581EB
+P 4100 6450
+F 0 "D3" V 4139 6332 50  0000 R CNN
+F 1 "LED" V 4048 6332 50  0000 R CNN
+F 2 "LED_THT:LED_D4.0mm" H 4100 6450 50  0001 C CNN
+F 3 "~" H 4100 6450 50  0001 C CNN
+	1    4100 6450
+	0    -1   -1   0
+$EndComp
+Wire Wire Line
+	3950 5700 4100 5700
+Wire Wire Line
+	4100 5850 4100 5700
+Connection ~ 4100 5700
+Wire Wire Line
+	4100 6150 4100 6300
+$Comp
+L Connector_Generic:Conn_01x02 J3
+U 1 1 6075E349
+P 4450 5900
+F 0 "J3" V 4322 5980 50  0000 L CNN
+F 1 "Conn_01x02" V 4413 5980 50  0000 L CNN
+F 2 "Connector_PinHeader_2.54mm:PinHeader_1x02_P2.54mm_Vertical" H 4450 5900 50  0001 C CNN
+F 3 "~" H 4450 5900 50  0001 C CNN
+	1    4450 5900
+	0    1    1    0
+$EndComp
+Wire Wire Line
+	4100 5700 4350 5700
+$Comp
+L power:GND #PWR0103
+U 1 1 6076295C
+P 3000 6700
+F 0 "#PWR0103" H 3000 6450 50  0001 C CNN
+F 1 "GND" H 3005 6527 50  0000 C CNN
+F 2 "" H 3000 6700 50  0001 C CNN
+F 3 "" H 3000 6700 50  0001 C CNN
+	1    3000 6700
+	1    0    0    -1
+$EndComp
+$Comp
+L power:GND #PWR0104
+U 1 1 60762E59
+P 3650 6700
+F 0 "#PWR0104" H 3650 6450 50  0001 C CNN
+F 1 "GND" H 3655 6527 50  0000 C CNN
+F 2 "" H 3650 6700 50  0001 C CNN
+F 3 "" H 3650 6700 50  0001 C CNN
+	1    3650 6700
+	1    0    0    -1
+$EndComp
+$Comp
+L power:GND #PWR0105
+U 1 1 607630CD
+P 4100 6700
+F 0 "#PWR0105" H 4100 6450 50  0001 C CNN
+F 1 "GND" H 4105 6527 50  0000 C CNN
+F 2 "" H 4100 6700 50  0001 C CNN
+F 3 "" H 4100 6700 50  0001 C CNN
+	1    4100 6700
+	1    0    0    -1
+$EndComp
+Wire Wire Line
+	3000 6100 3000 6700
+Wire Wire Line
+	3650 6000 3650 6700
+Wire Wire Line
+	4100 6600 4100 6700
+Wire Notes Line
+	5300 5400 5300 6950
+Wire Notes Line
+	5300 6950 1950 6950
+Wire Notes Line
+	1950 6950 1950 5400
+Wire Notes Line
+	1950 5400 5300 5400
+Text Notes 1950 5350 0    98   ~ 20
+Rectificador AC-DC\n
+$Comp
+L power:PWR_FLAG #FLG0103
+U 1 1 607743FC
+P 3000 5700
+F 0 "#FLG0103" H 3000 5775 50  0001 C CNN
+F 1 "PWR_FLAG" H 3000 5873 50  0000 C CNN
+F 2 "" H 3000 5700 50  0001 C CNN
+F 3 "~" H 3000 5700 50  0001 C CNN
+	1    3000 5700
+	1    0    0    -1
+$EndComp
 $EndSCHEMATC

Commit message: final desing with adc pin 24
Parts:
- removed R2: 1.5K, Resistor_THT:R_Axial_DIN0309_L9.0mm_D3.2mm_P5.08mm_Vertical, symbol Device:R
- added C2: 10uF, Capacitor_THT:CP_Radial_D5.0mm_P2.50mm, symbol Device:C
- added C3: 10uF, Capacitor_THT:CP_Radial_D5.0mm_P2.50mm, symbol Device:CP
- added D4: D, Diode_THT:D_A-405_P7.62mm_Horizontal, symbol Device:D
- added D5: LED, LED_THT:LED_D4.0mm, symbol Device:LED
- added R8, R9: 10k, Resistor_THT:R_Axial_DIN0309_L9.0mm_D3.2mm_P5.08mm_Vertical, symbol Device:R
- J4: footprint Connector_PinHeader_2.54mm:PinHeader_1x02_P2.54mm_Vertical -> TerminalBlock:TerminalBlock_bornier-2_P5.08mm
Connections:
- net 5v: now also R7.2, C3.1
- net Battery: now also R8.2
- net Fase: no longer U2.6
- net GND: now also C2.2, C3.2, R9.1
- net Neutro: now also U1.2
- net bridge: now also U2.6
- net at U2.1: now also D5.1 (K); no longer R5.1
- net at C1.1, D2.1 (K), U4.1 (VI): now also D4.1 (K)
- net at J3.2 (Pin_2), U4.3 (VO): now also D4.2 (A); no longer R7.2
- net Bat_adc: now reaches U3.7
- net Bat_adc: now also C2.1, R8.1, R9.2
- new net: D5.2 (A), R5.1
- no-connect marks 41 -> 40
Other:
- note added: "Converter AC-DC\n"
- note removed: "Rectificador AC-DC\n"
- moved on the sheet: BT1, C1, D1, D2, D3, J3, J4, L1, Q1, R6, R7, U2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
